File: MC34063_boost.kicad_sch (KiCad schematic)
At the start: 20 parts, among them U1 MC34063AP

Commit message: Fix: added indicating LED
Parts:
- added D?: RED, symbol Device:LED_Small
- added R?: 10k, symbol Device:R_Small
Connections:
- net GND: now also D?.1 (K)
- net at C4.1, C5.1, C6.1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: now also R?.1
- new net: D?.2 (A), R?.2
Other:
- moved on the sheet: TP4, TP5
Changed lines of the file:
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@@
   (junction (at 194.945 113.665) (diameter 0) (color 0 0 0 0)
   )
+  (junction (at 205.105 96.52) (diameter 0) (color 0 0 0 0)
+  )
   (junction (at 112.395 99.695) (diameter 0) (color 0 0 0 0)
   )
+  (junction (at 205.105 113.665) (diameter 0) (color 0 0 0 0)
+  )
   (junction (at 163.83 96.52) (diameter 0) (color 0 0 0 0)
   )
@@
   (junction (at 161.29 91.44) (diameter 0) (color 0 0 0 0)
   )
+  (wire (pts (xy 205.105 96.52) (xy 212.09 96.52))
+    (stroke (width 0) (type default) (color 0 0 0 0))
+  )
   (wire (pts (xy 161.29 85.09) (xy 161.29 88.9))
     (stroke (width 0) (type default) (color 0 0 0 0))
@@
     (stroke (width 0) (type default) (color 0 0 0 0))
   )
+  (wire (pts (xy 205.105 111.76) (xy 205.105 113.665))
+    (stroke (width 0) (type default) (color 0 0 0 0))
+  )
+  (wire (pts (xy 205.105 113.665) (xy 194.945 113.665))
+    (stroke (width 0) (type default) (color 0 0 0 0))
+  )
+  (wire (pts (xy 205.105 96.52) (xy 205.105 98.425))
+    (stroke (width 0) (type default) (color 0 0 0 0))
+  )
   (wire (pts (xy 131.445 88.9) (xy 129.54 88.9))
     (stroke (width 0) (type default) (color 0 0 0 0))
@@
     (stroke (width 0) (type default) (color 0 0 0 0))
   )
+  (wire (pts (xy 205.105 103.505) (xy 205.105 106.68))
+    (stroke (width 0) (type default) (color 0 0 0 0))
+  )
   (wire (pts (xy 112.395 88.9) (xy 112.395 92.075))
     (stroke (width 0) (type default) (color 0 0 0 0))
@@
     (stroke (width 0) (type default) (color 0 0 0 0))
   )
-  (wire (pts (xy 199.39 113.665) (xy 194.945 113.665))
+  (wire (pts (xy 212.09 113.665) (xy 205.105 113.665))
     (stroke (width 0) (type default) (color 0 0 0 0))
   )
@@
     (stroke (width 0) (type default) (color 0 0 0 0))
   )
-  (wire (pts (xy 194.945 96.52) (xy 199.39 96.52))
+  (wire (pts (xy 194.945 96.52) (xy 205.105 96.52))
     (stroke (width 0) (type default) (color 0 0 0 0))
   )
@@
     (pin "1")
   )
+  (symbol (lib_id "Device:R_Small") (at 205.105 100.965 0) (unit 1)
+    (in_bom yes) (on_board yes) (fields_autoplaced)
+    (property "Reference" "R?" (id 0) (at 207.01 99.6949 0)
+      (effects (font (size 1.27 1.27)) (justify left))
+    )
+    (property "Value" "10k" (id 1) (at 207.01 102.2349 0)
+      (effects (font (size 1.27 1.27)) (justify left))
+    )
+    (property "Footprint" "" (id 2) (at 205.105 100.965 0)
+      (effects (font (size 1.27 1.27)) hide)
+    )
+    (property "Datasheet" "~" (id 3) (at 205.105 100.965 0)
+      (effects (font (size 1.27 1.27)) hide)
+    )
+    (pin "1")
+    (pin "2")
+  )
   (symbol (lib_id "Device:L_Small") (at 156.845 93.98 90) (unit 1)
     (in_bom yes) (on_board yes)
@@
     (pin "2")
   )
-  (symbol (lib_id "Connector:TestPoint") (at 199.39 96.52 270) (unit 1)
-    (in_bom yes) (on_board yes)
-    (property "Reference" "TP4" (id 0) (at 202.565 98.425 90))
-    (property "Value" "Vout" (id 1) (at 206.375 96.52 90))
-    (property "Footprint" "TestPoint:TestPoint_Bridge_Pitch2.54mm_Drill1.0mm" (id 2) (at 199.39 101.6 0)
-      (effects (font (size 1.27 1.27)) hide)
-    )
-    (property "Datasheet" "~" (id 3) (at 199.39 101.6 0)
+  (symbol (lib_id "Connector:TestPoint") (at 212.09 96.52 270) (unit 1)
+    (in_bom yes) (on_board yes)
+    (property "Reference" "TP4" (id 0) (at 215.265 98.425 90))
+    (property "Value" "Vout" (id 1) (at 219.075 96.52 90))
+    (property "Footprint" "TestPoint:TestPoint_Bridge_Pitch2.54mm_Drill1.0mm" (id 2) (at 212.09 101.6 0)
+      (effects (font (size 1.27 1.27)) hide)
+    )
+    (property "Datasheet" "~" (id 3) (at 212.09 101.6 0)
       (effects (font (size 1.27 1.27)) hide)
     )
@@
     (pin "2")
   )
-  (symbol (lib_id "Connector:TestPoint") (at 199.39 113.665 270) (unit 1)
-    (in_bom yes) (on_board yes)
-    (property "Reference" "TP5" (id 0) (at 202.565 115.57 90))
-    (property "Value" "GND" (id 1) (at 206.375 113.665 90))
-    (property "Footprint" "TestPoint:TestPoint_Bridge_Pitch2.54mm_Drill1.0mm" (id 2) (at 199.39 118.745 0)
-      (effects (font (size 1.27 1.27)) hide)
-    )
-    (property "Datasheet" "~" (id 3) (at 199.39 118.745 0)
+  (symbol (lib_id "Connector:TestPoint") (at 212.09 113.665 270) (unit 1)
+    (in_bom yes) (on_board yes)
+    (property "Reference" "TP5" (id 0) (at 215.265 115.57 90))
+    (property "Value" "GND" (id 1) (at 219.075 113.665 90))
+    (property "Footprint" "TestPoint:TestPoint_Bridge_Pitch2.54mm_Drill1.0mm" (id 2) (at 212.09 118.745 0)
+      (effects (font (size 1.27 1.27)) hide)
+    )
+    (property "Datasheet" "~" (id 3) (at 212.09 118.745 0)
       (effects (font (size 1.27 1.27)) hide)
     )
@@
     )
     (pin "1")
+  )
+  (symbol (lib_id "Device:LED_Small") (at 205.105 109.22 90) (unit 1)
+    (in_bom yes) (on_board yes) (fields_autoplaced)
+    (property "Reference" "D?" (id 0) (at 207.01 107.8864 90)
+      (effects (font (size 1.27 1.27)) (justify right))
+    )
+    (property "Value" "RED" (id 1) (at 207.01 110.4264 90)
+      (effects (font (size 1.27 1.27)) (justify right))
+    )
+    (property "Footprint" "" (id 2) (at 205.105 109.22 90)
+      (effects (font (size 1.27 1.27)) hide)
+    )
+    (property "Datasheet" "~" (id 3) (at 205.105 109.22 90)
+      (effects (font (size 1.27 1.27)) hide)
+    )
+    (pin "1")
+    (pin "2")
   )
   (symbol (lib_id "Device:C_Small") (at 173.99 104.775 0) (unit 1)
@@
       (reference "D1") (unit 1) (value "1N4149") (footprint "Diode_THT:D_DO-35_SOD27_P7.62mm_Horizontal")
     )
+    (path "/b6f82404-04e2-4ad3-ba18-b5709d3e33d3"
+      (reference "D?") (unit 1) (value "RED") (footprint "")
+    )
     (path "/56f0ed1d-b051-4666-80cc-c23759923f3f"
       (reference "L1") (unit 1) (value "330u") (footprint "")
@@
       (reference "R5") (unit 1) (value "1k") (footprint "Resistor_THT:R_Axial_DIN0207_L6.3mm_D2.5mm_P10.16mm_Horizontal")
     )
+    (path "/13123ff5-bddf-4c72-a4f8-7ef1c921931b"
+      (reference "R?") (unit 1) (value "10k") (footprint "")
+    )
     (path "/db1c5641-736f-4d13-b04d-fb8d6ea2725e"

Commit message: Fix: changed LED colour to green
Parts:
- D?: value RED -> GREEN
Changed lines of the file:
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@@
       (effects (font (size 1.27 1.27)) (justify right))
     )
-    (property "Value" "RED" (id 1) (at 207.01 110.4264 90)
+    (property "Value" "GREEN" (id 1) (at 207.01 110.4264 90)
       (effects (font (size 1.27 1.27)) (justify right))
     )
@@
     )
     (path "/b6f82404-04e2-4ad3-ba18-b5709d3e33d3"
-      (reference "D?") (unit 1) (value "RED") (footprint "")
+      (reference "D?") (unit 1) (value "GREEN") (footprint "")
     )
     (path "/56f0ed1d-b051-4666-80cc-c23759923f3f"
